Commit message: [Update] Coppelia + Rviz2

File: src/irb_description/urdf/irb140.urdf (robot description, URDF)
Before this commit: robot abb_irb140, 9 links, 8 joints
Joints:
- joint joint_2: axis 0 1 0 -> 0 -1 0
- joint joint_3: axis 0 1 0 -> 0 -1 0
- joint joint_5: axis 0 1 0 -> 0 -1 0
- joint joint_6: axis 1 0 0 -> -1 0 0
